File: Calciumor_Under_Cover/Calciumor_Under_Cover.kicad_pcb (KiCad board)
At the start: 2 copper layers, 77 x 145 mm, 37 parts, among them J1 NeoPixel

Commit message: Core_rev1.0
Parts:
- added D33: SK6812MINI, LED_SMD:LED_SK6812MINI_PLCC4_3.5x3.5mm_P1.75mm, F.Cu at (59.6, 124.4)
- added D36: LED, LED_SMD:LED_0603_1608Metric, F.Cu at (72.0, 95.0)
- added D37: LED, LED_SMD:LED_0603_1608Metric, F.Cu at (72.0, 100.0)
- added D38: LED, LED_SMD:LED_0603_1608Metric, F.Cu at (72.0, 105.0)
- added D39: LED, LED_SMD:LED_0603_1608Metric, F.Cu at (72.0, 110.0)
- added D40: LED, LED_SMD:LED_0603_1608Metric, F.Cu at (72.0, 115.0)
- added D41: LED, LED_SMD:LED_0603_1608Metric, F.Cu at (72.0, 120.0)
- added D42: LED, LED_SMD:LED_0603_1608Metric, F.Cu at (72.0, 125.0)
- added D43: LED, LED_SMD:LED_0603_1608Metric, F.Cu at (72.0, 130.0)
- added D44: LED, LED_SMD:LED_0603_1608Metric, F.Cu at (72.0, 135.0)
- added D45: LED, LED_SMD:LED_0603_1608Metric, F.Cu at (72.0, 140.0)
- added D46: LED, LED_SMD:LED_0603_1608Metric, F.Cu at (72.0, 145.0)
- added D47: LED, LED_SMD:LED_0603_1608Metric, F.Cu at (72.0, 150.0)
- added D48: LED, LED_SMD:LED_0603_1608Metric, F.Cu at (72.0, 155.0)
- added D49: LED, LED_SMD:LED_0603_1608Metric, F.Cu at (72.0, 160.0)
- added D50: LED, LED_SMD:LED_0603_1608Metric, F.Cu at (72.0, 165.0)
- added D51: LED, LED_SMD:LED_0603_1608Metric, F.Cu at (72.0, 170.0)
- added D52: LED, LED_SMD:LED_0603_1608Metric, F.Cu at (72.0, 175.0)
- added D53: LED, LED_SMD:LED_0603_1608Metric, F.Cu at (76.0, 178.0)
- added D54: LED, LED_SMD:LED_0603_1608Metric, F.Cu at (81.0, 178.0)
- added D55: LED, LED_SMD:LED_0603_1608Metric, F.Cu at (86.0, 178.0)
- added D56: LED, LED_SMD:LED_0603_1608Metric, F.Cu at (91.0, 178.0)
- added D57: LED, LED_SMD:LED_0603_1608Metric, F.Cu at (96.0, 178.0)
- added D58: LED, LED_SMD:LED_0603_1608Metric, F.Cu at (101.0, 178.0)
- added D59: LED, LED_SMD:LED_0603_1608Metric, F.Cu at (106.0, 178.0)
- added D60: LED, LED_SMD:LED_0603_1608Metric, F.Cu at (111.0, 178.0)
- added D61: LED, LED_SMD:LED_0603_1608Metric, F.Cu at (116.0, 178.0)
- added D62: LED, LED_SMD:LED_0603_1608Metric, F.Cu at (121.0, 178.0)
- added D63: LED, LED_SMD:LED_0603_1608Metric, F.Cu at (126.0, 178.0)
- added D64: LED, LED_SMD:LED_0603_1608Metric, F.Cu at (131.0, 178.0)
- added D65: LED, LED_SMD:LED_0603_1608Metric, F.Cu at (136.0, 178.0)
- added D66: LED, LED_SMD:LED_0603_1608Metric, F.Cu at (141.0, 178.0)
- added D67: LED, LED_SMD:LED_0603_1608Metric, F.Cu at (145.0, 175.0)
- added D68: LED, LED_SMD:LED_0603_1608Metric, F.Cu at (145.0, 170.0)
- added D69: LED, LED_SMD:LED_0603_1608Metric, F.Cu at (145.0, 165.0)
- added D70: LED, LED_SMD:LED_0603_1608Metric, F.Cu at (145.0, 160.0)
- added D71: LED, LED_SMD:LED_0603_1608Metric, F.Cu at (145.0, 155.0)
- added D72: LED, LED_SMD:LED_0603_1608Metric, F.Cu at (145.0, 150.0)
- added D73: LED, LED_SMD:LED_0603_1608Metric, F.Cu at (145.0, 145.0)
- added D74: LED, LED_SMD:LED_0603_1608Metric, F.Cu at (145.0, 140.0)
- added D75: LED, LED_SMD:LED_0603_1608Metric, F.Cu at (145.0, 135.0)
- added D76: LED, LED_SMD:LED_0603_1608Metric, F.Cu at (145.0, 130.0)
- added D77: LED, LED_SMD:LED_0603_1608Metric, F.Cu at (145.0, 125.0)
- added D78: LED, LED_SMD:LED_0603_1608Metric, F.Cu at (145.0, 120.0)
- added D79: LED, LED_SMD:LED_0603_1608Metric, F.Cu at (145.0, 115.0)
- added D80: LED, LED_SMD:LED_0603_1608Metric, F.Cu at (145.0, 110.0)
- added D81: LED, LED_SMD:LED_0603_1608Metric, F.Cu at (145.0, 105.0)
- added D82: LED, LED_SMD:LED_0603_1608Metric, F.Cu at (145.0, 100.0)
- added D83: LED, LED_SMD:LED_0603_1608Metric, F.Cu at (145.0, 95.0)
- added D84: LED, LED_SMD:LED_0603_1608Metric, F.Cu at (145.0, 90.0)
- added J2: NeoPixel, Connector_JST:JST_PH_S4B-PH-SM4-TB_1x04-1MP_P2.00mm_Horizontal, B.Cu at (139.0, 80.0)
- added R1: 470, Resistor_SMD:R_1206_3216Metric, F.Cu at (80.0, 171.5)
- D1, D10, D11, D12, D13, D14, D15, D16, D17, D18, D19, D2, D20, D21, D22, D23, D24, D25, D26, D27, D28, D29, D3, D30, D31, D32, D34, D4, D5, D6, D7, D8, D9: value WS2812B -> SK6812MINI; footprint LED_SMD:LED_WS2812B_PLCC4_5.0x5.0mm_P3.2mm -> LED_SMD:LED_SK6812MINI_PLCC4_3.5x3.5mm_P1.75mm
- D35: value WS2812B -> LED; footprint LED_SMD:LED_WS2812B_PLCC4_5.0x5.0mm_P3.2mm -> LED_SMD:LED_0603_1608Metric
- G***: moved to B.Cu
- moved D4 107.6 mm to (31.5, 119.3), turned to 0 degrees
- moved G*** 101.4 mm to (106.0, 163.0), turned to 180 degrees
- moved D8 99.5 mm to (38.5, 104.2), turned to 0 degrees
- moved G*** 98.6 mm to (81.0, 163.0), turned to 180 degrees
- moved D7 97.3 mm to (31.5, 134.5), turned to 0 degrees
- moved D16 96.4 mm to (45.5, 109.2), turned to 0 degrees
- moved D30 96.2 mm to (59.6, 109.2), turned to 0 degrees
- moved D29 92.5 mm to (59.6, 104.2), turned to 0 degrees
- moved D15 89.4 mm to (45.5, 104.2), turned to 0 degrees
- moved D35 88.8 mm to (72.0, 90.0), turned to 0 degrees
- moved D3 88.0 mm to (31.5, 114.3), turned to 0 degrees
- moved D14 83.5 mm to (38.5, 134.5)
- moved D32 80.0 mm to (59.6, 119.3), turned to 0 degrees
- moved D11 79.5 mm to (38.5, 119.3)
- moved D6 78.2 mm to (31.5, 129.4), turned to 0 degrees
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Connections:
- D1 pad 1: +5V -> Net-(D1-DOUT)
- D1 pad 2: Net-(D1-DOUT) -> GND
- D1 pad 3: GND -> /RGB
- D1 pad 4: /RGB -> +5V
- D10 pad 1: +5V -> Net-(D10-DOUT)
- D10 pad 2: Net-(D10-DOUT) -> GND
- D10 pad 3: GND -> /D4
- D10 pad 4: Net-(D10-DIN) -> +5V
- D11 pad 1: +5V -> Net-(D11-DOUT)
- D11 pad 2: Net-(D10-DIN) -> GND
- D11 pad 3: GND -> Net-(D10-DOUT)
- D11 pad 4: Net-(D11-DIN) -> +5V
- D12 pad 1: +5V -> /D7
- D12 pad 2: Net-(D12-DOUT) -> GND
- D12 pad 3: GND -> Net-(D12-DIN)
- D12 pad 4: Net-(D12-DIN) -> +5V
- D13 pad 1: +5V -> Net-(D12-DIN)
- D13 pad 2: Net-(D12-DIN) -> GND
- D13 pad 3: GND -> Net-(D13-DIN)
- D13 pad 4: Net-(D13-DIN) -> +5V
- D14 pad 1: +5V -> Net-(D13-DIN)
- D14 pad 2: Net-(D13-DIN) -> GND
- D14 pad 3: GND -> /D4
- D14 pad 4: Net-(D14-DIN) -> +5V
- D15 pad 1: +5V -> /D7
- D15 pad 2: Net-(D11-DIN) -> GND
- D15 pad 3: GND -> Net-(D11-DOUT)
- D15 pad 4: Net-(D15-DIN) -> +5V
- D16 pad 1: +5V -> /D4
- D16 pad 2: Net-(D14-DIN) -> GND
- D16 pad 3: GND -> /D3
- D16 pad 4: Net-(D16-DIN) -> +5V
- D17 pad 1: +5V -> /D14
- D17 pad 2: Net-(D17-DOUT) -> GND
- D17 pad 3: GND -> Net-(D17-DIN)
- D17 pad 4: Net-(D17-DIN) -> +5V
- D18 pad 1: +5V -> Net-(D17-DIN)
- D18 pad 2: Net-(D18-DOUT) -> GND
- D18 pad 3: GND -> Net-(D18-DIN)
- D18 pad 4: Net-(D17-DOUT) -> +5V
- D19 pad 1: +5V -> Net-(D18-DIN)
- D19 pad 2: Net-(D19-DOUT) -> GND
- D19 pad 3: GND -> /D11
- D19 pad 4: Net-(D18-DOUT) -> +5V
- D2 pad 1: +5V -> Net-(D2-DOUT)
- D2 pad 2: Net-(D2-DOUT) -> GND
- D2 pad 3: GND -> Net-(D1-DOUT)
- D2 pad 4: Net-(D1-DOUT) -> +5V
- D20 pad 1: +5V -> Net-(D20-DOUT)
- D20 pad 2: Net-(D20-DOUT) -> GND
- D20 pad 3: GND -> /D7
- D20 pad 4: Net-(D12-DOUT) -> +5V
- D21 pad 1: +5V -> Net-(D21-DOUT)
- D21 pad 2: Net-(D21-DOUT) -> GND
- D21 pad 3: GND -> Net-(D20-DOUT)
- D21 pad 4: Net-(D20-DOUT) -> +5V
- D22 pad 1: +5V -> /D10
- D22 pad 2: Net-(D22-DOUT) -> GND
- D22 pad 3: GND -> Net-(D21-DOUT)
- D22 pad 4: Net-(D21-DOUT) -> +5V
- D23 pad 1: +5V -> /D11
- D23 pad 2: Net-(D23-DOUT) -> GND
- D23 pad 3: GND -> /D10
- D23 pad 4: Net-(D23-DIN) -> +5V
- D24 pad 1: +5V -> Net-(D24-DOUT)
- D24 pad 2: Net-(D23-DIN) -> GND
- D24 pad 3: GND -> /D7
- D24 pad 4: Net-(D24-DIN) -> +5V
- D25 pad 1: +5V -> Net-(D25-DOUT)
- D25 pad 2: Net-(D24-DIN) -> GND
- D25 pad 3: GND -> Net-(D24-DOUT)
- D25 pad 4: Net-(D25-DIN) -> +5V
- D26 pad 1: +5V -> /D14
- D26 pad 2: Net-(D26-DOUT) -> GND
- D26 pad 3: GND -> Net-(D26-DIN)
- D26 pad 4: Net-(D26-DIN) -> +5V
- D27 pad 1: +5V -> Net-(D26-DIN)
- D27 pad 2: Net-(D26-DIN) -> GND
- D27 pad 3: GND -> Net-(D27-DIN)
- D27 pad 4: Net-(D27-DIN) -> +5V
- D28 pad 1: +5V -> Net-(D27-DIN)
- D28 pad 2: Net-(D27-DIN) -> GND
- D28 pad 3: GND -> /D11
- D28 pad 4: Net-(D28-DIN) -> +5V
- D29 pad 1: +5V -> /D10
- D29 pad 2: Net-(D25-DIN) -> GND
- D29 pad 3: GND -> Net-(D25-DOUT)
- D29 pad 4: Net-(D19-DOUT) -> +5V
- D3 pad 1: +5V -> Net-(D3-DOUT)
- D3 pad 2: Net-(D3-DOUT) -> GND
- D3 pad 3: GND -> Net-(D2-DOUT)
- D3 pad 4: Net-(D2-DOUT) -> +5V
- D30 pad 1: +5V -> /D11
- D30 pad 2: Net-(D28-DIN) -> GND
- D30 pad 3: GND -> /D10
- D30 pad 4: Net-(D22-DOUT) -> +5V
- D31 pad 1: +5V -> Net-(D31-DOUT)
- D31 pad 2: Net-(D31-DOUT) -> GND
- D31 pad 3: GND -> /D14
- D31 pad 4: Net-(D23-DOUT) -> +5V
- D32 pad 1: +5V -> unconnected-(D32-DOUT-Pad1)
- D32 pad 2: unconnected-(D32-DOUT-Pad2) -> GND
- D32 pad 3: GND -> Net-(D31-DOUT)
- D32 pad 4: Net-(D31-DOUT) -> +5V
- D34 pad 1: +5V -> unconnected-(D34-DOUT-Pad1)
- D34 pad 2: Net-(D34-DOUT) -> GND
- D34 pad 3: GND -> Net-(D33-DOUT)
- D34 pad 4: Net-(D26-DOUT) -> +5V
- D35 pad 1: +5V -> /LED_R
- D35 pad 2: unconnected-(D35-DOUT-Pad2) -> /LED
- D4 pad 1: +5V -> /D3
- D4 pad 2: Net-(D15-DIN) -> GND
- D4 pad 3: GND -> Net-(D3-DOUT)
- D4 pad 4: Net-(D3-DOUT) -> +5V
- D5 pad 1: +5V -> Net-(D5-DOUT)
- D5 pad 2: Net-(D5-DOUT) -> GND
- D5 pad 3: GND -> /RGB
- D5 pad 4: /RGB -> +5V
- D6 pad 1: +5V -> Net-(D6-DOUT)
- D6 pad 2: Net-(D6-DOUT) -> GND
- D6 pad 3: GND -> Net-(D5-DOUT)
- D6 pad 4: Net-(D5-DOUT) -> +5V
- D7 pad 1: +5V -> Net-(D7-DOUT)
- D7 pad 2: Net-(D7-DOUT) -> GND
- D7 pad 3: GND -> Net-(D6-DOUT)
- D7 pad 4: Net-(D6-DOUT) -> +5V
- D8 pad 1: +5V -> /D3
- D8 pad 2: Net-(D16-DIN) -> GND
- D8 pad 3: GND -> Net-(D7-DOUT)
- D8 pad 4: Net-(D7-DOUT) -> +5V
- D9 pad 1: +5V -> /D4
- D9 pad 2: Net-(D17-DIN) -> GND
- D9 pad 3: GND -> /D3
- D9 pad 4: Net-(D10-DOUT) -> +5V
Routing:
- net +5V: track 551.2 -> 16.5 mm, vias 0 -> 2
- net /LED: track 0.00 -> 339.0 mm, vias 0 -> 3
- net /RGB: track 27.9 -> 69.5 mm, vias 0 -> 2
- net Net-(D22-DOUT): track 40.6 -> 0.00 mm
- net Net-(D28-DIN): track 37.2 -> 0.00 mm
- net Net-(D16-DIN): track 36.4 -> 0.00 mm
- net Net-(D14-DIN): track 36.2 -> 0.00 mm
- net Net-(D15-DIN): track 34.1 -> 0.00 mm
- net Net-(D26-DOUT): track 32.2 -> 0.00 mm
- net Net-(D19-DOUT): track 31.6 -> 0.00 mm
- net Net-(D23-DOUT): track 29.3 -> 0.00 mm
- net Net-(D12-DOUT): track 27.1 -> 0.00 mm
- net Net-(D11-DIN): track 26.7 -> 0.00 mm
- net Net-(D25-DIN): track 26.4 -> 0.00 mm
- net Net-(D34-DOUT): track 25.0 -> 0.00 mm
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- added copper zone on F.Cu, net /LED_R
Other:
- board size 77 x 145 mm -> 77 x 105.6 mm

Commit message: Under cover completed
Parts:
- removed J2: NeoPixel, Connector_JST:JST_PH_S4B-PH-SM4-TB_1x04-1MP_P2.00mm_Horizontal
- added H1: MountingHole, MountingHole:MountingHole_2.2mm_M2, F.Cu at (89.5, 103.5)
- added H2: MountingHole, MountingHole:MountingHole_2.2mm_M2, F.Cu at (127.5, 103.5)
- added H3: MountingHole, MountingHole:MountingHole_2.2mm_M2, F.Cu at (89.5, 141.5)
- added H4: MountingHole, MountingHole:MountingHole_2.2mm_M2, F.Cu at (127.5, 141.5)
- D1, D10, D11, D12, D13, D14, D15, D16, D17, D18, D19, D2, D20, D21, D22, D23, D24, D25, D26, D27, D28, D29, D3, D30, D31, D32, D33, D34, D4, D5, D6, D7, D8, D9: value SK6812MINI -> WS2812B; footprint LED_SMD:LED_SK6812MINI_PLCC4_3.5x3.5mm_P1.75mm -> LED_SMD:LED_WS2812B_PLCC4_5.0x5.0mm_P3.2mm
- moved D4 107.6 mm to (137.0, 98.0), turned to 180 degrees
- moved D8 99.5 mm to (137.0, 90.0), turned to 180 degrees
- moved D29 98.6 mm to (140.5, 160.5), turned to 90 degrees
- moved D7 97.3 mm to (118.0, 90.0), turned to 180 degrees
- moved D15 96.7 mm to (140.5, 122.5), turned to 90 degrees
- moved D30 89.9 mm to (133.5, 160.5), turned to 90 degrees
- moved D16 89.0 mm to (133.5, 122.5), turned to 90 degrees
- moved D3 88.0 mm to (118.0, 98.0), turned to 180 degrees
- moved D14 83.5 mm to (118.0, 109.0)
- moved D32 79.7 mm to (118.0, 173.5), turned to 180 degrees
- moved D11 79.5 mm to (118.0, 117.0)
- moved D6 78.2 mm to (99.0, 90.0), turned to 180 degrees
- moved D25 74.5 mm to (118.0, 155.0)
- moved D19 73.4 mm to (118.0, 136.0), turned to 180 degrees
- moved D22 69.6 mm to (118.0, 128.0), turned to 180 degrees
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Connections:
- D1 pad 1: Net-(D1-DOUT) -> +5V
- D1 pad 2: GND -> Net-(D1-DOUT)
- D1 pad 3: /RGB -> GND
- D1 pad 4: +5V -> /RGB
- D10 pad 1: Net-(D10-DOUT) -> +5V
- D10 pad 2: GND -> Net-(D10-DOUT)
- D10 pad 3: /D4 -> GND
- D10 pad 4: +5V -> Net-(D10-DIN)
- D11 pad 1: Net-(D11-DOUT) -> +5V
- D11 pad 2: GND -> Net-(D10-DIN)
- D11 pad 3: Net-(D10-DOUT) -> GND
- D11 pad 4: +5V -> /D4
- D12 pad 1: /D7 -> +5V
- D12 pad 2: GND -> /D7
- D12 pad 3: Net-(D12-DIN) -> GND
- D12 pad 4: +5V -> /D6
- D13 pad 1: Net-(D12-DIN) -> +5V
- D13 pad 2: GND -> /D6
- D13 pad 3: Net-(D13-DIN) -> GND
- D13 pad 4: +5V -> /D5
- D14 pad 1: Net-(D13-DIN) -> +5V
- D14 pad 2: GND -> /D5
- D14 pad 3: /D4 -> GND
- D14 pad 4: +5V -> /D4
- D15 pad 1: /D7 -> +5V
- D15 pad 2: GND -> /D4
- D15 pad 3: Net-(D11-DOUT) -> GND
- D15 pad 4: +5V -> /D3
- D16 pad 1: /D4 -> +5V
- D16 pad 2: GND -> /D4
- D16 pad 3: /D3 -> GND
- D16 pad 4: +5V -> /D3
- D17 pad 1: /D14 -> +5V
- D17 pad 2: GND -> Net-(D17-DOUT)
- D17 pad 3: Net-(D17-DIN) -> GND
- D17 pad 4: +5V -> /D7
- D18 pad 1: Net-(D17-DIN) -> +5V
- D18 pad 2: GND -> Net-(D18-DOUT)
- D18 pad 3: Net-(D18-DIN) -> GND
- D18 pad 4: +5V -> Net-(D17-DOUT)
- D19 pad 1: Net-(D18-DIN) -> +5V
- D19 pad 2: GND -> /D10
- D19 pad 3: /D11 -> GND
- D19 pad 4: +5V -> Net-(D18-DOUT)
- D2 pad 1: Net-(D2-DOUT) -> +5V
- D2 pad 2: GND -> Net-(D2-DOUT)
- D2 pad 3: Net-(D1-DOUT) -> GND
- D2 pad 4: +5V -> Net-(D1-DOUT)
- D20 pad 1: Net-(D20-DOUT) -> +5V
- D20 pad 2: GND -> /D8
- D20 pad 3: /D7 -> GND
- D20 pad 4: +5V -> /D7
- D21 pad 1: Net-(D21-DOUT) -> +5V
- D21 pad 2: GND -> /D9
- D21 pad 3: Net-(D20-DOUT) -> GND
- D21 pad 4: +5V -> /D8
- D22 pad 1: /D10 -> +5V
- D22 pad 2: GND -> /D10
- D22 pad 3: Net-(D21-DOUT) -> GND
- D22 pad 4: +5V -> /D9
- D23 pad 1: /D11 -> +5V
- D23 pad 2: GND -> /D14
- D23 pad 3: /D10 -> GND
- D23 pad 4: +5V -> Net-(D23-DIN)
- D24 pad 1: Net-(D24-DOUT) -> +5V
- D24 pad 2: GND -> Net-(D23-DIN)
- D24 pad 3: /D7 -> GND
- D24 pad 4: +5V -> Net-(D24-DIN)
- D25 pad 1: Net-(D25-DOUT) -> +5V
- D25 pad 2: GND -> Net-(D24-DIN)
- D25 pad 3: Net-(D24-DOUT) -> GND
- D25 pad 4: +5V -> /D11
- D26 pad 1: /D14 -> +5V
- D26 pad 2: GND -> /D14
- D26 pad 3: Net-(D26-DIN) -> GND
- D26 pad 4: +5V -> /D13
- D27 pad 1: Net-(D26-DIN) -> +5V
- D27 pad 2: GND -> /D13
- D27 pad 3: Net-(D27-DIN) -> GND
- D27 pad 4: +5V -> /D12
- D28 pad 1: Net-(D27-DIN) -> +5V
- D28 pad 2: GND -> /D12
- D28 pad 3: /D11 -> GND
- D28 pad 4: +5V -> /D11
- D29 pad 1: /D10 -> +5V
- D29 pad 2: GND -> /D11
- D29 pad 3: Net-(D25-DOUT) -> GND
- D29 pad 4: +5V -> /D10
- D3 pad 1: Net-(D3-DOUT) -> +5V
- D3 pad 2: GND -> Net-(D3-DOUT)
- D3 pad 3: Net-(D2-DOUT) -> GND
- D3 pad 4: +5V -> Net-(D2-DOUT)
- D30 pad 1: /D11 -> +5V
- D30 pad 2: GND -> /D11
- D30 pad 3: /D10 -> GND
- D30 pad 4: +5V -> /D10
- D31 pad 1: Net-(D31-DOUT) -> +5V
- D31 pad 2: GND -> Net-(D31-DOUT)
- D31 pad 3: /D14 -> GND
- D31 pad 4: +5V -> /D14
- D32 pad 1: unconnected-(D32-DOUT-Pad1) -> +5V
- D32 pad 2: GND -> unconnected-(D32-DOUT-Pad2)
- D32 pad 3: Net-(D31-DOUT) -> GND
- D32 pad 4: +5V -> Net-(D31-DOUT)
- D33 pad 1: Net-(D33-DOUT) -> +5V
- D33 pad 2: GND -> /D15
- D33 pad 3: /D14 -> GND
- D33 pad 4: +5V -> /D14
- D34 pad 1: unconnected-(D34-DOUT-Pad1) -> +5V
- D34 pad 2: GND -> unconnected-(D34-DOUT-Pad2)
- D34 pad 3: Net-(D33-DOUT) -> GND
- D34 pad 4: +5V -> /D15
- D4 pad 1: /D3 -> +5V
- D4 pad 2: GND -> /D3
- D4 pad 3: Net-(D3-DOUT) -> GND
- D4 pad 4: +5V -> Net-(D3-DOUT)
- D5 pad 1: Net-(D5-DOUT) -> +5V
- D5 pad 2: GND -> /D0
- D5 pad 3: /RGB -> GND
- D5 pad 4: +5V -> /RGB
- D6 pad 1: Net-(D6-DOUT) -> +5V
- D6 pad 2: GND -> /D1
- D6 pad 3: Net-(D5-DOUT) -> GND
- D6 pad 4: +5V -> /D0
- D7 pad 1: Net-(D7-DOUT) -> +5V
- D7 pad 2: GND -> /D2
- D7 pad 3: Net-(D6-DOUT) -> GND
- D7 pad 4: +5V -> /D1
- D8 pad 1: /D3 -> +5V
- D8 pad 2: GND -> /D3
- D8 pad 3: Net-(D7-DOUT) -> GND
- D8 pad 4: +5V -> /D2
- D9 pad 1: /D4 -> +5V
- D9 pad 2: GND -> /D7
- D9 pad 3: /D3 -> GND
- D9 pad 4: +5V -> Net-(D10-DOUT)
Routing:
- net +5V: track 16.5 -> 543.0 mm, vias 2 -> 0
- net /RGB: track 69.5 -> 145.8 mm, vias 2 -> 0
- net /D4: track 1.95 -> 63.4 mm
- net /D11: track 1.60 -> 60.8 mm
- net /D10: track 0.00 -> 57.5 mm
- net /D3: track 0.00 -> 54.2 mm
- net /D14: track 1.90 -> 40.4 mm
- net /D7: track 0.00 -> 37.9 mm
- net Net-(D31-DOUT): track 0.00 -> 25.0 mm
- net /D15: track 0.00 -> 25.0 mm
- net Net-(D3-DOUT): track 0.00 -> 15.5 mm
- net /D2: track 0.00 -> 15.5 mm
- net Net-(D24-DIN): track 0.00 -> 15.5 mm
- net Net-(D23-DIN): track 0.00 -> 15.5 mm
- net Net-(D2-DOUT): track 0.00 -> 15.5 mm
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Other:
- board size 77 x 105.6 mm -> 77 x 96.5 mm
- board text added: "Calciumor Revision 1.0 Developed by Chrodream"
